File: Sensor Node/pcb layout/LoRa Water Quality Management System Sensor Node/rp2350_layout.kicad_sch (KiCad schematic)
At the start: 28 parts, among them J1 Conn_01x03, J2 Conn_01x02, U1 RP2350_60QFN, U2 W25Q128JVSIQ TR, Y1 ABM8-272-T3

Commit message: Add finalized schematics for sx1262 and SPI flash.
Parts:
- renumbered C13 to C10, C1 to C11, C11 to C13, C4 to C14, C5 to C15, C6 to C16, C7 to C17, C8 to C18, C9 to C19, C10 to C20, C14 to C5, C15 to C6, C16 to C7, C2 to C8, C3 to C9, J2 to J3, J1 to J4, R6 to R10, R3 to R5, R2 to R6, R1 to R7, R4 to R8, R5 to R9, U2 to U1, U1 to U2

Commit message: Finalize first draft schematic capture, assign all footprints, and begin preliminary PCB layout.
Parts:
- C14: renamed from C5; footprint (none) -> Capacitor_SMD:C_0603_1608Metric_Pad1.08x0.95mm_HandSolder
- C15: renamed from C6; footprint (none) -> Capacitor_SMD:C_0603_1608Metric_Pad1.08x0.95mm_HandSolder
- C16: renamed from C7; footprint (none) -> Capacitor_SMD:C_0603_1608Metric_Pad1.08x0.95mm_HandSolder
- C17: renamed from C8; footprint (none) -> Capacitor_SMD:C_0603_1608Metric_Pad1.08x0.95mm_HandSolder
- C18: renamed from C9; footprint (none) -> Capacitor_SMD:C_0603_1608Metric_Pad1.08x0.95mm_HandSolder
- C19: renamed from C10; footprint (none) -> Capacitor_SMD:C_0603_1608Metric_Pad1.08x0.95mm_HandSolder
- C20: renamed from C11; footprint (none) -> Capacitor_SMD:C_0603_1608Metric_Pad1.08x0.95mm_HandSolder
- C21: renamed from C12; footprint (none) -> Capacitor_SMD:C_0603_1608Metric_Pad1.08x0.95mm_HandSolder
- C22: renamed from C13; footprint (none) -> Capacitor_SMD:C_0603_1608Metric_Pad1.08x0.95mm_HandSolder
- C23: renamed from C14; footprint (none) -> Capacitor_SMD:C_0603_1608Metric_Pad1.08x0.95mm_HandSolder
- C24: renamed from C15; footprint (none) -> Capacitor_SMD:C_0603_1608Metric_Pad1.08x0.95mm_HandSolder
- C25: renamed from C16; footprint (none) -> Capacitor_SMD:C_0603_1608Metric_Pad1.08x0.95mm_HandSolder
- C26: renamed from C17; footprint (none) -> Capacitor_SMD:C_0603_1608Metric_Pad1.08x0.95mm_HandSolder
- C27: renamed from C18; footprint (none) -> Capacitor_SMD:C_0603_1608Metric_Pad1.08x0.95mm_HandSolder
- C28: renamed from C19; footprint (none) -> Capacitor_SMD:C_0603_1608Metric_Pad1.08x0.95mm_HandSolder
- C29: renamed from C20; footprint (none) -> Capacitor_SMD:C_0603_1608Metric_Pad1.08x0.95mm_HandSolder
- J8: renamed from J3; footprint (none) -> Connector_PinHeader_2.54mm:PinHeader_1x02_P2.54mm_Vertical
- J9: renamed from J4; footprint (none) -> Connector_PinHeader_2.54mm:PinHeader_1x03_P2.54mm_Vertical
- L1: footprint (none) -> LWQMS:AOTA-B201610S3R3-101-T
- R14: renamed from R5; footprint (none) -> Resistor_SMD:R_0603_1608Metric_Pad0.98x0.95mm_HandSolder
- R15: renamed from R6; footprint (none) -> Resistor_SMD:R_0603_1608Metric_Pad0.98x0.95mm_HandSolder
- R16: renamed from R7; footprint (none) -> Resistor_SMD:R_0603_1608Metric_Pad0.98x0.95mm_HandSolder
- R17: renamed from R8; footprint (none) -> Resistor_SMD:R_0603_1608Metric_Pad0.98x0.95mm_HandSolder
- R18: renamed from R9; footprint (none) -> Resistor_SMD:R_0603_1608Metric_Pad0.98x0.95mm_HandSolder
- R19: renamed from R10; footprint (none) -> Resistor_SMD:R_0603_1608Metric_Pad0.98x0.95mm_HandSolder
- U7: renamed from U1; footprint SOIC_208MIL_WIN -> LWQMS:SOIC_208MIL_WIN-M
- U8: renamed from U2; footprint RP2350_60QFN_minimal:RP2350-QFN-60-1EP_7x7_P0.4mm_EP3.4x3.4mm_ThermalVias -> LWQMS:RP2350-QFN-60-1EP_7x7_P0.4mm_EP3.4x3.4mm_ThermalVias
- Y1: footprint (none) -> LWQMS:ABM8-272-T3

Commit message: Add power supply PCB layout
Parts:
- renumbered R14 to R17, R15 to R18, R16 to R19, R17 to R20, R18 to R21, R19 to R22
Changed lines of the file:
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@@
 		(on_board yes)
 		(dnp no)
-		(property "Reference" "R14"
+		(property "Reference" "R17"
 			(at 49.784 184.15 0)
 			(effects
@@
 			(project ""
 				(path "/f090528b-8c52-4bf9-a2b8-0c17aa5e5727/8ed505b3-7460-4c84-b5db-8c51c81aa9b0"
-					(reference "R14")
+					(reference "R17")
 					(unit 1)
 				)
@@
 		(on_board yes)
 		(dnp no)
-		(property "Reference" "R15"
+		(property "Reference" "R18"
 			(at 66.04 165.1 0)
 			(effects
@@
 			(project ""
 				(path "/f090528b-8c52-4bf9-a2b8-0c17aa5e5727/8ed505b3-7460-4c84-b5db-8c51c81aa9b0"
-					(reference "R15")
+					(reference "R18")
 					(unit 1)
 				)
@@
 		(on_board yes)
 		(dnp no)
-		(property "Reference" "R19"
+		(property "Reference" "R22"
 			(at 304.8 111.506 90)
 			(effects
@@
 			(project "LoRa Water Quality Management System Sensor Node"
 				(path "/f090528b-8c52-4bf9-a2b8-0c17aa5e5727/8ed505b3-7460-4c84-b5db-8c51c81aa9b0"
-					(reference "R19")
+					(reference "R22")
 					(unit 1)
 				)
@@
 		(on_board yes)
 		(dnp no)
-		(property "Reference" "R18"
+		(property "Reference" "R21"
 			(at 304.8 104.648 90)
 			(effects
@@
 			(project ""
 				(path "/f090528b-8c52-4bf9-a2b8-0c17aa5e5727/8ed505b3-7460-4c84-b5db-8c51c81aa9b0"
-					(reference "R18")
+					(reference "R21")
 					(unit 1)
 				)
@@
 		(on_board yes)
 		(dnp no)
-		(property "Reference" "R16"
+		(property "Reference" "R19"
 			(at 196.85 89.154 90)
 			(effects
@@
 			(project ""
 				(path "/f090528b-8c52-4bf9-a2b8-0c17aa5e5727/8ed505b3-7460-4c84-b5db-8c51c81aa9b0"
-					(reference "R16")
+					(reference "R19")
 					(unit 1)
 				)
@@
 		(on_board yes)
 		(dnp no)
-		(property "Reference" "R17"
+		(property "Reference" "R20"
 			(at 215.9 160.274 90)
 			(effects
@@
 			(project "LoRa Water Quality Management System Sensor Node"
 				(path "/f090528b-8c52-4bf9-a2b8-0c17aa5e5727/8ed505b3-7460-4c84-b5db-8c51c81aa9b0"
-					(reference "R17")
-					(unit 1)
-				)
+					(reference "R20")
+					(unit 1)
+				)

Commit message: finalize RP2350 layout (mostly)
Other:
- note added: "One Decoupling Capacitor for pins 1, 11, 20, 30, 38, (44,45), 54"
- note removed: "One Decoupling Capacitor for pins 1, 11, 20, 30, 38, 54 (pin 45 may need one as well, not shown in reference design)"
Changed lines of the file:
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@@
 		)
 	)
-	(text "One Decoupling Capacitor for pins 1, 11, 20, 30, 38, 54\n(pin 45 may need one as well, not shown in reference design)"
+	(text "One Decoupling Capacitor for pins 1, 11, 20, 30, 38, (44,45), 54"
 		(exclude_from_sim no)
 		(at 344.17 54.864 0)
