File: Sensor Node/pcb layout/LoRa Water Quality Management System Sensor Node/LoRa Water Quality Management System Sensor Node.kicad_pcb (KiCad board)
At the start: 2 copper layers, 100 x 100 mm, 94 parts, among them J1 PxC 1757255, J2 PxC 1757242, J3 Conn_Coaxial, J4 PxC 1757255, J5 PxC 1757255, J6 USB_B, J7 Conn_Coaxial, J8 Conn_01x02, J9 Conn_01x03, SW1 Tactile Pushbutton, U1 TMUX1309, U10 TPS631010YBGR, U11 LMV324, U12 MCP4651T-503E/ML, U13 MCP4651T-503E/ML, U2 LSF0102, U3 TMUX1309, U4 Core1262 HF, U5 MX25L3233FM2I-08Q, U6 MCP3425Axx-xCH, U7 W25Q128JVSIQ TR, U8 RP2350_60QFN, U9 TPS631010YBGR, Y1 ABM8-272-T3

Commit message: Add power supply PCB layout
Parts:
- added D4: 5.1-5.7V, Diode_SMD:D_SOD-128, F.Cu at (-72.6, 60.2)
- added R30: 10k, Resistor_SMD:R_0603_1608Metric_Pad0.98x0.95mm_HandSolder, F.Cu at (-32.1, 68.0)
- added R31: 10k, Resistor_SMD:R_0603_1608Metric_Pad0.98x0.95mm_HandSolder, F.Cu at (-32.1, 70.5)
- added R32: 10k, Resistor_SMD:R_0603_1608Metric_Pad0.98x0.95mm_HandSolder, F.Cu at (-32.1, 73.0)
- D1: value BAT54C -> B240AE-13; footprint Package_TO_SOT_SMD:TSOT-23_HandSoldering -> Diode_SMD:D_SMA_Handsoldering
- D2: value 3.3-3.7V -> B240AE-13; footprint Diode_SMD:D_SOD-128 -> Diode_SMD:D_SMA_Handsoldering
- D3: value 5.1-5.7V -> 3.3-3.7V
- R10: value 10k -> 100R
- R11: value 10k -> 200k
- R14: value 1k -> 10k
- R16: value 33R -> 10k
- R18: value 27R -> 10k
- R19: value 27R -> 33R
- R20: value 10k -> 1k
- R21, R22: value 10k -> 27R
- R3: value 511k -> 10k
- R4: value 91k -> 10k
- R5: value 806k -> 10k
- R6: value 91k -> 511k
- R7: value 100R -> 91k
- R8: value 200k -> 806k
- R9: value 10k -> 91k
- moved D3 270.4 mm to (-72.6, 56.1)
- moved SW1 244.6 mm to (-60.9, 60.2)
- moved C1 239.4 mm to (172.6, 51.9), turned to 180 degrees
- moved C2 238.2 mm to (172.7, 66.0), turned to 180 degrees
- moved U8 235.2 mm to (-58.7, 86.1)
- moved Y1 234.8 mm to (-74.5, 87.5)
- moved C3 234.6 mm to (167.6, 55.2)
- moved C4 233.2 mm to (167.5, 69.1)
- moved U7 233.2 mm to (-57.6, 68.0)
- moved R7 229.5 mm to (169.2, 51.9)
- moved R6 226.9 mm to (167.4, 53.4)
- moved U12 226.4 mm to (-46.4, 67.7)
- moved U13 226.4 mm to (-46.4, 74.6)
- moved R8 225.4 mm to (167.3, 67.6)
- moved J8 224.1 mm to (-56.4, 74.0)
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Connections:
- D1 pad 1: /V_{BATT} -> /V_{IN}
- D1 pad 2: /USB_VBUS -> /V_{BATT}
- D2 pad 1: +3V3 -> /V_{IN}
- D2 pad 2: GND -> /USB_VBUS
- D3 pad 1: +5V -> +3V3
- J3 pad 1: /PH_IN -> /PH_RAW
- J3 pad 2: GND -> /PH_GND
- J4 pad 1: +5V -> /RTD_SEN
- J4 pad 2: /EXTRA_IN -> unconnected-(J4-Pin_2-Pad2)
- J4 pad 3: /EXTRA_GND -> /RTD_GND
- J5 pad 1: /RTD_SEN -> +5V
- J5 pad 2: unconnected-(J5-Pin_2-Pad2) -> /EXTRA_IN
- J5 pad 3: /RTD_GND -> /EXTRA_GND
- R10 pad 2: /I2C_SCL_{0}_5V -> /RTD_SEN
- R11 pad 1: +3V3 -> +5V
- R11 pad 2: /MCU/~{RESET} -> Net-(U2-EN)
- R12 pad 1: +3V3 -> +5V
- R12 pad 2: Net-(U5-~{HOLD}) -> /I2C_SDA_{0}_5V
- R13 pad 1: +3V3 -> +5V
- R13 pad 2: Net-(U5-~{WP}) -> /I2C_SCL_{0}_5V
- R14 pad 1: Net-(J8-Pin_1) -> +3V3
- R14 pad 2: /MCU/QSPI_SS -> /MCU/~{RESET}
- R15 pad 2: /MCU/QSPI_SS -> Net-(U5-~{HOLD})
- R16 pad 2: /MCU/VREG_AVDD -> Net-(U5-~{WP})
- R17 pad 1: Net-(U8-XOUT) -> Net-(J8-Pin_1)
- R17 pad 2: Net-(C16-Pad2) -> /MCU/QSPI_SS
- R18 pad 1: Net-(U8-USB_DP) -> +3V3
- R18 pad 2: /MCU/USB_D+ -> /MCU/QSPI_SS
- R19 pad 1: Net-(U8-USB_DM) -> +3V3
- R19 pad 2: /MCU/USB_D- -> /MCU/VREG_AVDD
- R20 pad 1: /Software-Defined Instrumentation Amplifier/IN+ -> Net-(U8-XOUT)
- R20 pad 2: Net-(U11D-+) -> Net-(C16-Pad2)
- R21 pad 1: /Software-Defined Instrumentation Amplifier/V_{offset+} -> Net-(U8-USB_DP)
- R21 pad 2: Net-(U11D-+) -> /MCU/USB_D+
- R22 pad 1: /Software-Defined Instrumentation Amplifier/V_{offset-} -> Net-(U8-USB_DM)
- R22 pad 2: Net-(U11D--) -> /MCU/USB_D-
- R23 pad 1: Net-(U11D--) -> /Software-Defined Instrumentation Amplifier/IN+
- R23 pad 2: /Software-Defined Instrumentation Amplifier/V_SENSOR_WITH_DC_OFFSET -> Net-(U11D-+)
- R24 pad 1: Net-(R24-Pad1) -> /Software-Defined Instrumentation Amplifier/V_{offset+}
- R24 pad 2: /Software-Defined Instrumentation Amplifier/RGain+ -> Net-(U11D-+)
- R25 pad 1: /Software-Defined Instrumentation Amplifier/RGain- -> /Software-Defined Instrumentation Amplifier/V_{offset-}
- R25 pad 2: Net-(R25-Pad2) -> Net-(U11D--)
- R26 pad 1: Net-(R24-Pad1) -> Net-(U11D--)
- R26 pad 2: Net-(U11C--) -> /Software-Defined Instrumentation Amplifier/V_SENSOR_WITH_DC_OFFSET
- R27 pad 1: Net-(R25-Pad2) -> Net-(R27-Pad1)
- R27 pad 2: Net-(U11C-+) -> /Software-Defined Instrumentation Amplifier/RGain+
- R28 pad 1: Net-(U11C--) -> /Software-Defined Instrumentation Amplifier/RGain-
- R28 pad 2: /Software-Defined Instrumentation Amplifier/OUT -> Net-(R28-Pad2)
- R29 pad 1: Net-(U11C-+) -> Net-(R27-Pad1)
- R29 pad 2: GND -> Net-(U11C--)
- R3 pad 2: /Buck-Boost Regulator (TPS631010YBGR) Layout/FB -> /PH_IN
- R4 pad 1: /Buck-Boost Regulator (TPS631010YBGR) Layout/FB -> /PH_RAW
- R4 pad 2: GND -> /PH_IN
- R5 pad 1: +5V -> /PH_GND
- R5 pad 2: /Buck-Boost Regulator (TPS631010YBGR) Layout1/FB -> /PH_IN
- R6 pad 1: /Buck-Boost Regulator (TPS631010YBGR) Layout1/FB -> +3V3
- R6 pad 2: GND -> /Buck-Boost Regulator (TPS631010YBGR) Layout/FB
- R7 pad 1: +5V -> /Buck-Boost Regulator (TPS631010YBGR) Layout/FB
- R7 pad 2: /RTD_SEN -> GND
- R8 pad 2: Net-(U2-EN) -> /Buck-Boost Regulator (TPS631010YBGR) Layout1/FB
- R9 pad 1: +5V -> /Buck-Boost Regulator (TPS631010YBGR) Layout1/FB
- R9 pad 2: /I2C_SDA_{0}_5V -> GND
- U1 pad 14: unconnected-(U1-S1A-Pad14) -> /PH_GND
- U11 pad 1: Net-(R24-Pad1) -> Net-(R27-Pad1)
- U11 pad 7: Net-(R25-Pad2) -> Net-(R28-Pad2)
- U3 pad 5: GND -> /PH_GND
Routing:
- net /V_{BATT}: track 0.00 -> 11.5 mm
- net /USB_VBUS: track 0.00 -> 9.20 mm
- net /Buck-Boost Regulator (TPS631010YBGR) Layout1/FB: track 0.00 -> 4.95 mm
- net /Buck-Boost Regulator (TPS631010YBGR) Layout/FB: track 0.00 -> 4.95 mm
- net GND: vias 0 -> 24
- net /V_{IN}: vias 0 -> 16
- net +5V: vias 0 -> 29
- net +3V3: vias 0 -> 14
- added copper zone on F.Cu, net +3V3
- added copper zone on In1.Cu, net +3V3
- added copper zone on F.Cu, net +5V
- added copper zone on In1.Cu, net +5V
- added copper zone on F.Cu, net /V_{IN}
- added copper zone on F.Cu, net GND
- added copper zone on In2.Cu, net GND
- added copper zone on F.Cu, net Net-(U10-LX1)
- added copper zone on F.Cu, net Net-(U10-LX2)
- added copper zone on F.Cu, net Net-(U9-LX1)
- added copper zone on F.Cu, net Net-(U9-LX2)
Other:
- board size 100 x 100 mm -> 100 x 75 mm
- copper layers 2 -> 4

Commit message: Begin RP2350 PCB layout
Parts:
- moved R21 208.2 mm to (139.9, 41.3)
- moved R22 208.2 mm to (139.9, 43.8)
- moved C20 205.7 mm to (129.6, 52.3), turned to -90 degrees
- moved C18 200.9 mm to (125.4, 52.6)
- moved C17 200.5 mm to (125.4, 54.1)
- moved C21 199.9 mm to (125.1, 67.2), turned to -90 degrees
- moved C25 199.4 mm to (129.4, 63.0)
- moved C16 197.8 mm to (123.6, 71.1), turned to 90 degrees
- moved L1 196.6 mm to (124.5, 50.8)
- moved R19 196.3 mm to (129.6, 48.7), turned to -90 degrees
- moved Y1 194.1 mm to (118.9, 72.0)
- moved C23 192.7 mm to (122.2, 51.6), turned to 90 degrees
- moved C26 191.7 mm to (121.6, 65.8), turned to -90 degrees
- moved C19 191.3 mm to (116.1, 58.5), turned to 180 degrees
- moved C15 191.0 mm to (116.8, 71.1), turned to -90 degrees
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Routing:
- net +3V3: track 0.00 -> 22.6 mm, vias 14 -> 23
- net /USB_VBUS: track 9.20 -> 24.9 mm
- net Net-(U8-XIN): track 0.00 -> 13.2 mm
- net GND: track 0.00 -> 10.0 mm, vias 24 -> 36
- net /MCU/VREG_AVDD: track 0.00 -> 8.28 mm
- net +1V1: track 0.00 -> 7.57 mm, vias 0 -> 3
- net /LoRa_~{RESET}: track 0.00 -> 6.34 mm
- net /I2C_SDA_{0}: track 0.00 -> 5.92 mm
- net /I2C_SCL_{0}: track 0.00 -> 5.90 mm
- net /LoRa_BUSY: track 0.00 -> 5.87 mm
- net Net-(C16-Pad2): track 0.00 -> 4.48 mm
- net /MCU/GPIO3: track 0.00 -> 4.30 mm
- net /LoRa_IRQ: track 0.00 -> 4.27 mm
- net /UART_RX_{0}: track 0.00 -> 4.24 mm
- net /UART_TX_{0}: track 0.00 -> 4.22 mm
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- added copper zone on B.Cu, net +1V1
- added copper zone on F.Cu, net +1V1
- added copper zone on In2.Cu, net +3V3
- added copper zone on B.Cu, net +5V
- added copper zone on In2.Cu, net +5V
- added copper zone on F.Cu, net /MCU/VREG_LX
- added copper zone on In1.Cu, net GND
- removed copper zone on In1.Cu, net +3V3
- removed copper zone on In1.Cu, net +5V
- removed copper zone on In2.Cu, net GND

Commit message: finalize RP2350 layout (mostly)
Parts:
- moved C14 259.7 mm to (185.2, 52.3)
- moved R17 250.9 mm to (185.2, 53.9), turned to 180 degrees
- moved J8 244.0 mm to (187.0, 56.9), turned to -90 degrees
- moved R18 234.9 mm to (168.8, 51.3), turned to -90 degrees
- moved U7 233.9 mm to (175.9, 54.2)
- moved C29 230.5 mm to (160.4, 72.1), turned to -90 degrees
- moved C22 227.1 mm to (157.1, 72.1), turned to -90 degrees
- moved C24 225.5 mm to (155.6, 72.1), turned to -90 degrees
- moved U4 174.3 mm to (109.3, 60.1), turned to 90 degrees
- moved J9 133.4 mm to (72.2, 67.7), turned to 90 degrees
- moved U5 128.6 mm to (74.0, 74.9)
- moved C23 43.9 mm to (165.2, 60.3), turned to 0 degrees
- moved C28 43.8 mm to (159.9, 57.6), turned to 90 degrees
- moved L1 43.3 mm to (165.1, 65.9), turned to -90 degrees
- moved R19 43.2 mm to (166.5, 71.1), turned to 180 degrees
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Connections:
- net /MCU/USB_D+ renamed /USB_D+
- net /MCU/USB_D- renamed /USB_D-
- U8 pad 12: /~{SENSOR_EN} -> /LoRa_IRQ
- U8 pad 13: /SENSOR_SEL_0 -> /MCU/GPIO9
- U8 pad 14: /SENSOR_SEL_1 -> /MCU/GPIO10
- U8 pad 33: /MCU/GPIO21 -> /~{SENSOR_EN}
- U8 pad 34: /MCU/GPIO22 -> /SENSOR_SEL_0
- U8 pad 35: /MCU/GPIO23 -> /SENSOR_SEL_1
Routing:
- net /MCU/QSPI_SS: track 0.00 -> 30.8 mm
- net /USB_D+: track 0.00 -> 30.4 mm
- net /MCU/QSPI_SD3: track 0.00 -> 30.3 mm
- net /USB_D-: track 0.00 -> 28.9 mm
- net /MCU/QSPI_SCLK: track 0.00 -> 27.9 mm
- net /MCU/QSPI_SD0: track 0.00 -> 24.8 mm
- net +3V3: track 22.6 -> 44.4 mm, vias 23 -> 24
- net /MCU/QSPI_SD1: track 0.00 -> 17.7 mm
- net /MCU/QSPI_SD2: track 0.00 -> 17.3 mm
- net GND: track 10.0 -> 18.4 mm, vias 36 -> 42
- net +1V1: track 7.57 -> 14.7 mm, vias 3 -> 4
- net Net-(U8-USB_DP): track 0.00 -> 6.06 mm
- net /MCU/SWCLK: track 0.00 -> 5.70 mm
- net Net-(U8-USB_DM): track 0.00 -> 5.69 mm
- net /MCU/SWD: track 0.00 -> 5.23 mm
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
Commit message: Finalize most routing, preliminary RF design (fencing/stitching vias) RF transmission line trace, etc.
Parts:
- moved D3 259.2 mm to (185.9, 75.2), turned to -90 degrees
- moved D4 255.4 mm to (182.3, 75.2), turned to -90 degrees
- moved R3 228.3 mm to (185.4, 84.4), turned to 90 degrees
- moved R4 226.3 mm to (183.8, 84.4), turned to 90 degrees
- moved R5 224.1 mm to (182.2, 84.4), turned to 90 degrees
- moved SW1 210.6 mm to (148.0, 33.5), turned to 180 degrees
- moved C5 208.6 mm to (160.5, 79.3), turned to 180 degrees
- moved C6 203.9 mm to (155.6, 82.2), turned to -90 degrees
- moved U1 193.0 mm to (147.5, 88.2), turned to 90 degrees
- moved R11 192.8 mm to (154.0, 82.2), turned to 90 degrees
- moved C7 191.7 mm to (142.6, 86.9), turned to 180 degrees
- moved U2 190.6 mm to (155.3, 79.1), turned to 180 degrees
- moved R12 190.1 mm to (151.8, 80.1), turned to 90 degrees
- moved C9 189.6 mm to (149.5, 43.9), turned to 90 degrees
- moved R14 187.7 mm to (157.0, 37.1), turned to -90 degrees
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Connections:
- net /I2C_SCL_{0}_5V renamed /I2C_SCL_{1}_5V
- net /I2C_SDA_{0}_5V renamed /I2C_SDA_{1}_5V
- net Net-(J7-In) renamed /RF_OUT
- U13 pad 10: /Software-Defined Instrumentation Amplifier/RGain+ -> Net-(U13-P0B)
- U13 pad 7: Net-(U13-P0W) -> Net-(U13-P0B)
- U13 pad 9: Net-(U13-P0W) -> Net-(U13-P0B)
- U2 pad 3: /I2C_SDA_{0} -> /I2C_SDA_{1}
- U2 pad 4: /I2C_SCL_{0} -> /I2C_SCL_{1}
- U8 pad 10: /LoRa_~{RESET} -> /MCU/GPIO7
- U8 pad 13: /MCU/GPIO9 -> /LoRa_BUSY
- U8 pad 14: /MCU/GPIO10 -> /LoRa_~{RESET}
- U8 pad 15: /MCU/GPIO11 -> /LoRa_CS
- U8 pad 28: /LoRa_CS -> /MCU/GPIO17
- U8 pad 32: /~{FLASH_CS} -> /MCU/GPIO20
- U8 pad 4: /LoRa_IRQ -> /MCU/GPIO2
- U8 pad 40: /MCU/GPIO26_ADC0 -> /I2C_SDA_{1}
- U8 pad 41: /MCU/GPIO27_ADC1 -> /I2C_SCL_{1}
- U8 pad 7: /I2C_SDA_{0} -> /MCU/GPIO4
- U8 pad 8: /I2C_SCL_{0} -> /MCU/GPIO5
- U8 pad 9: /LoRa_BUSY -> /~{FLASH_CS}
Routing:
- net /PH_GND: track 0.00 -> 60.1 mm, vias 0 -> 2
- net /I2C_SDA_{1}_5V: track 0.00 -> 57.5 mm, vias 0 -> 3
- net /PH_IN: track 0.00 -> 55.8 mm
- net /I2C_SCL_{1}_5V: track 0.00 -> 54.6 mm, vias 0 -> 4
- net /~{SENSOR_EN}: track 0.00 -> 54.2 mm, vias 0 -> 3
- net /EXTRA_GND: track 0.00 -> 45.7 mm, vias 0 -> 2
- net /SENSOR_SEL_0: track 0.00 -> 43.2 mm, vias 0 -> 4
- net /SENSOR_SEL_1: track 0.00 -> 42.2 mm, vias 0 -> 4
- net /MCU/~{RESET}: track 4.86 -> 45.4 mm, vias 0 -> 2
- net /EXTRA_IN: track 0.00 -> 39.8 mm, vias 0 -> 2
- net /TURB_IN: track 0.00 -> 39.6 mm, vias 0 -> 1
- net /RTD_GND: track 0.00 -> 39.5 mm
- net /Software-Defined Instrumentation Amplifier/IN-: track 0.00 -> 33.7 mm
- net /TURB_GND: track 0.00 -> 33.0 mm, vias 0 -> 2
- net +3V3: track 44.4 -> 70.9 mm, vias 24 -> 32
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
Commit message: Improved RF routing, import all 3D models.
Parts:
- added C32: 100n, Capacitor_SMD:C_0603_1608Metric_Pad1.08x0.95mm_HandSolder, F.Cu at (108.7, 81.4)
- added D5: ESDARF02-1BU2CK, Diode_SMD:D_0201_0603Metric_Pad0.64x0.40mm_HandSolder, F.Cu at (114.1, 34.6)
- added G*** (x2): LOGO, LWQMS:psh, F.Cu at (0.00, 0.00)
- J7: value Conn_Coaxial -> SMA-J-P-X-RA-TH1; footprint Connector_Coaxial:SMA_Amphenol_901-143_Horizontal -> LWQMS:SAMTEC_SMA-J-P-X-RA-TH1
- moved C13 45.0 mm to (120.8, 92.1), turned to 90 degrees
- moved C12 44.8 mm to (119.3, 92.1), turned to 90 degrees
- moved C10 44.6 mm to (133.3, 64.9)
- moved U4 31.9 mm to (134.9, 40.1)
- moved C11 28.7 mm to (117.8, 92.1), turned to 90 degrees
- moved R15 11.0 mm to (144.8, 56.3)
- moved C9 10.3 mm to (148.1, 54.1), turned to 0 degrees
- moved R16 6.40 mm to (141.0, 43.1)
- moved J7 5.97 mm to (114.7, 30.0), turned to -90 degrees
- moved U5 2.80 mm to (143.2, 50.5), turned to -90 degrees
- moved D3 1.98 mm to (186.0, 77.2)
- moved D4 1.98 mm to (182.5, 77.1)
- moved R28 1.74 mm to (108.8, 83.0)
- moved R27 1.74 mm to (108.8, 79.7)
- moved R29 1.69 mm to (108.7, 78.2)
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Routing:
- net /SPI_SCK_{0}: track 0.00 -> 68.8 mm
- net /SPI_MISO_{0}: track 0.00 -> 63.7 mm
- net /SPI_MOSI_{0}: track 0.00 -> 61.6 mm
- net /LoRa_CS: track 0.00 -> 47.0 mm, vias 0 -> 2
- net /LoRa_IRQ: track 3.69 -> 44.3 mm, vias 0 -> 2
- net /LoRa_~{RESET}: track 3.27 -> 38.5 mm, vias 0 -> 2
- net /LoRa_BUSY: track 3.38 -> 37.2 mm, vias 0 -> 2
- net /RF_OUT: track 23.0 -> 10.2 mm
- net Net-(U4-DIO2): track 0.00 -> 12.6 mm
- net /UART_RX_{0}: track 4.24 -> 0.00 mm
- net /UART_TX_{0}: track 4.22 -> 0.00 mm
- net /MCU/QSPI_SCLK: track 30.6 -> 27.2 mm
- net /~{FLASH_CS}: track 23.4 -> 20.9 mm
- net Net-(U11C--): track 17.9 -> 15.3 mm
- net Net-(R27-Pad1): track 7.97 -> 5.92 mm
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Other:
- board text added: "BOOTSEL"
- board text added: "EXTRA"
- board text added: "JST DEBUG"
- board text added: "PT100 RTD"
- board text added: "RESET"
- board text added: "SWCLK GND SWD"
- board text added: "TURB."
- board text added: "pH"

Commit message: Improve RF routing and noise immunity. Add copper pours on top and bottom layer with ample stitching vias. Add TVS diodes for ESD protection and testpoints for hardware debugging.
Parts:
- removed G*** (x2): LOGO, LWQMS:psh
- removed the REF** at (195.5, 30.5)
- removed the REF** at (195.5, 95.5)
- removed the REF** at (105.5, 95.5)
- added D10: ESDZV5HS-1BF4, Diode_SMD:D_0201_0603Metric_Pad0.64x0.40mm_HandSolder, F.Cu at (192.2, 49.1)
- added D5: ESDZV5HS-1BF4, Diode_SMD:D_0201_0603Metric_Pad0.64x0.40mm_HandSolder, F.Cu at (178.8, 49.2)
- added D6: ESDZV5HS-1BF4, Diode_SMD:D_0201_0603Metric_Pad0.64x0.40mm_HandSolder, F.Cu at (189.2, 52.7)
- added D9: ESDARF02-1BU2CK, Diode_SMD:D_0201_0603Metric_Pad0.64x0.40mm_HandSolder, F.Cu at (162.3, 50.1)
- added J6: Conn_01x02, Connector_PinHeader_2.54mm:PinHeader_1x02_P2.54mm_Vertical, F.Cu at (143.1, 36.5)
- added REF**: MountingHole_3.2mm_M3_DIN965_Pad, MountingHole:MountingHole_3.2mm_M3_DIN965_Pad, F.Cu at (105.5, 95.5)
- added REF**: MountingHole_3.2mm_M3_DIN965_Pad, MountingHole:MountingHole_3.2mm_M3_DIN965_Pad, F.Cu at (195.5, 95.5)
- added REF**: MountingHole_3.2mm_M3_DIN965_Pad, MountingHole:MountingHole_3.2mm_M3_DIN965_Pad, F.Cu at (195.5, 30.6)
- added TP1: TestPoint, TestPoint:TestPoint_Pad_D1.5mm, F.Cu at (192.5, 85.5)
- added TP10: TestPoint, TestPoint:TestPoint_Pad_D1.5mm, F.Cu at (110.8, 86.4)
- added TP11: TestPoint, TestPoint:TestPoint_Pad_D1.5mm, F.Cu at (118.5, 75.6)
- added TP12: TestPoint_Small, TestPoint:TestPoint_Pad_D1.5mm, F.Cu at (124.3, 74.1)
- added TP13: TestPoint_Small, TestPoint:TestPoint_Pad_D1.5mm, F.Cu at (121.4, 74.1)
- added TP14: TestPoint_Small, TestPoint:TestPoint_Pad_D1.5mm, F.Cu at (115.3, 75.5)
- added TP15: TestPoint, TestPoint:TestPoint_Pad_D1.5mm, F.Cu at (138.2, 74.0)
- added TP16: TestPoint, TestPoint:TestPoint_Pad_D1.5mm, F.Cu at (135.4, 74.1)
- added TP2: TestPoint, TestPoint:TestPoint_Pad_D1.5mm, F.Cu at (132.6, 74.1)
- added TP3: TestPoint, TestPoint:TestPoint_Pad_D1.5mm, F.Cu at (143.3, 81.1)
- added TP4: TestPoint, TestPoint:TestPoint_Pad_D1.5mm, F.Cu at (180.8, 38.1)
- added TP5: TestPoint, TestPoint:TestPoint_Pad_D1.5mm, F.Cu at (129.8, 74.1)
- added TP6: TestPoint, TestPoint:TestPoint_Pad_D1.5mm, F.Cu at (146.6, 81.1)
- added TP7: TestPoint, TestPoint:TestPoint_Pad_D1.5mm, F.Cu at (182.4, 46.9)
- added TP8: TestPoint, TestPoint:TestPoint_Pad_D1.5mm, F.Cu at (182.4, 42.7)
- added TP9: TestPoint, TestPoint:TestPoint_Pad_D1.5mm, F.Cu at (127.0, 74.1)
- R12, R13: value 10k -> 4k
- moved R17 8.38 mm to (137.6, 32.9), turned to -90 degrees
- moved J9 4.45 mm to (143.1, 32.8), turned to -90 degrees
- moved C5 2.20 mm to (159.2, 80.2), turned to 90 degrees
- moved R19 0.25 mm to (166.2, 71.1)
- moved D7 0.20 mm to (114.3, 34.5)
- renumbered C32 to C31, C31 to C32, D5 to D7, J9 to J10, J6 to J7, J7 to J8, J8 to J9
Connections:
- REF** pad 1: (no net) -> GND
Routing:
- net /UART_RX_{0}: track 0.00 -> 33.2 mm, vias 0 -> 1
- net /UART_TX_{0}: track 0.00 -> 31.4 mm, vias 0 -> 1
- net GND: track 42.2 -> 56.2 mm, vias 293 -> 778
- net /RTD_SEN: track 17.8 -> 28.5 mm, vias 0 -> 2
- net /MCU/QSPI_SS: track 48.7 -> 59.1 mm
- net /TURB_IN: track 39.6 -> 48.7 mm
- net /PH_RAW: track 3.52 -> 12.3 mm
- net /Software-Defined Instrumentation Amplifier/V_{offset-}: track 10.8 -> 18.6 mm
- net /Software-Defined Instrumentation Amplifier/V_{offset+}: track 12.6 -> 20.3 mm
- net /Software-Defined Instrumentation Amplifier/OUT: track 8.15 -> 15.8 mm, vias 0 -> 2
- net /Software-Defined Instrumentation Amplifier/IN+: track 7.31 -> 14.6 mm
- net /I2C_SDA_{1}_5V: track 56.0 -> 61.2 mm
- net /I2C_SCL_{1}_5V: track 53.7 -> 58.7 mm
- net +5V: track 22.3 -> 27.2 mm
- net /PH_IN: track 55.8 -> 60.2 mm, vias 0 -> 2
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- added copper zone on B.Cu, net GND
Other:
- board text added: "RX TX"
- board text removed: "BOOTSEL"
