File: Sensor Node/pcb layout/LoRa Water Quality Management System Sensor Node/LoRa Water Quality Management System Sensor Node.kicad_pcb (KiCad board)
At the start: 4 copper layers, 130 x 80 mm, 162 parts, among them J1 OQ0332510000G, J10 Conn_01x03, J2 OQ0232510000G, J3 CONBNC002, J4 OQ0332510000G, J5 OQ0332510000G, J6 Conn_01x02, J7 USB_B, J8 SMA-J-P-X-RA-TH1, J9 Conn_01x02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

Commit message: Implemented RDT3.0 for LoRa data transfer.
Parts:
- R30: value 3k -> 10k
- R31: value 1k -> 10k
- R32, R34: value 30k -> 4.99k
- R33: value 60k -> 10k
- R8: value 100R -> 4.7k
Changed lines of the file:
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@@
 			)
 		)
-		(property "Value" "1k"
+		(property "Value" "10k"
 			(at 0 1.65 90)
 			(layer "F.Fab")
@@
 			)
 		)
-		(property "Value" "100R"
+		(property "Value" "4.7k"
 			(at 0 1.65 0)
 			(layer "F.Fab")
@@
 			)
 		)
-		(property "Value" "3k"
+		(property "Value" "10k"
 			(at 0 1.65 90)
 			(layer "F.Fab")
@@
 			)
 		)
-		(property "Value" "60k"
+		(property "Value" "10k"
 			(at 0 1.65 90)
 			(layer "F.Fab")
@@
 			)
 		)
-		(property "Value" "30k"
+		(property "Value" "4.99k"
 			(at 0 1.65 0)
 			(layer "F.Fab")
@@
 			)
 		)
-		(property "Value" "30k"
+		(property "Value" "4.99k"
 			(at 0 1.65 90)
 			(layer "F.Fab")
@@
 	)
 	(zone
-		(net 51)
-		(net_name "/SPI_SCK_{0}")
-		(layer "F.Cu")
-		(name "$teardrop_padvia$")
-		(hatch none 0.1)
-		(priority 30003)
-		(attr
-			(teardrop
-				(type padvia)
-			)
-		)
-		(connect_pads yes
-			(clearance 0)
-		)
-		(min_thickness 0.0254)
-		(filled_areas_thickness no)
-		(fill yes
-			(thermal_gap 0.5)
-			(thermal_bridge_width 0.5)
-			(island_removal_mode 1)
-			(island_area_min 10)
-		)
-		(polygon
-			(pts
-				(xy 148.00947 92.57447) (xy 148.20947 92.57447) (xy 148.408666 92.2224) (xy 148.10947 91.46347)
-				(xy 147.810274 92.2224)
-			)
-		)
-	)
-	(zone
-		(net 51)
-		(net_name "/SPI_SCK_{0}")
-		(layer "F.Cu")
-		(name "$teardrop_padvia$")
-		(hatch none 0.1)
-		(priority 30005)
-		(attr
-			(teardrop
-				(type padvia)
-			)
-		)
-		(connect_pads yes
-			(clearance 0)
-		)
-		(min_thickness 0.0254)
-		(filled_areas_thickness no)
-		(fill yes
-			(thermal_gap 0.5)
-			(thermal_bridge_width 0.5)
-			(island_removal_mode 1)
-			(island_area_min 10)
-		)
-		(polygon
-			(pts
-				(xy 148.20947 90.35447) (xy 148.00947 90.35447) (xy 147.810274 90.70654) (xy 148.10947 91.46547)
-				(xy 148.408666 90.70654)
-			)
-		)
-	)
-	(zone
 		(net 3)
 		(net_name "+3V3")
@@
 	)
 	(zone
-		(net 54)
-		(net_name "/SPI_MISO_{0}")
+		(net 55)
+		(net_name "/SPI_MOSI_{0}")
 		(layer "F.Cu")
 		(name "$teardrop_padvia$")
 		(hatch none 0.1)
-		(priority 30004)
+		(priority 30007)
 		(attr
 			(teardrop
@@
 		(polygon
 			(pts
-				(xy 149.27947 85.36447) (xy 149.47947 85.36447) (xy 149.678666 85.0124) (xy 149.37947 84.25347)
-				(xy 149.080274 85.0124)
+				(xy 146.73947 92.57447) (xy 146.93947 92.57447) (xy 147.138666 92.2224) (xy 146.83947 91.46347)
+				(xy 146.540274 92.2224)
 			)
 		)
@@
 	)
 	(zone
+		(net 54)
+		(net_name "/SPI_MISO_{0}")
+		(layer "F.Cu")
+		(name "$teardrop_padvia$")
+		(hatch none 0.1)
+		(priority 30005)
+		(attr
+			(teardrop
+				(type padvia)
+			)
+		)
+		(connect_pads yes
+			(clearance 0)
+		)
+		(min_thickness 0.0254)
+		(filled_areas_thickness no)
+		(fill yes
+			(thermal_gap 0.5)
+			(thermal_bridge_width 0.5)
+			(island_removal_mode 1)
+			(island_area_min 10)
+		)
+		(polygon
+			(pts
+				(xy 149.27947 85.36447) (xy 149.47947 85.36447) (xy 149.678666 85.0124) (xy 149.37947 84.25347)
+				(xy 149.080274 85.0124)
+			)
+		)
+	)
+	(zone
 		(net 3)
 		(net_name "+3V3")
@@
 	)
 	(zone
-		(net 92)
-		(net_name "Net-(U9-L1)")
+		(net 51)
+		(net_name "/SPI_SCK_{0}")
 		(layer "F.Cu")
-		(name "U9_L1")
-		(hatch edge 0.5)
-		(priority 5)
+		(name "$teardrop_padvia$")
+		(hatch none 0.1)
+		(priority 30003)
+		(attr
+			(teardrop
+				(type padvia)
+			)
+		)
 		(connect_pads yes
-			(clearance 0.15)
+			(clearance 0)
 		)
-		(min_thickness 0.25)
+		(min_thickness 0.0254)
 		(filled_areas_thickness no)
 		(fill yes
 			(thermal_gap 0.5)
 			(thermal_bridge_width 0.5)
+			(island_removal_mode 1)
+			(island_area_min 10)
 		)
 		(polygon
 			(pts
-				(xy 169.69947 71.89947) (xy 169.69947 71.40947) (xy 171.40947 71.40947) (xy 172.42947 70.38947)
-				(xy 175.26697 70.38947) (xy 175.41947 70.54197) (xy 175.41947 71.75947) (xy 175.27947 71.89947)
+				(xy 148.00947 92.57447) (xy 148.20947 92.57447) (xy 148.408666 92.2224) (xy 148.10947 91.46347)
+				(xy 147.810274 92.2224)
 			)
 		)
 	)
 	(zone
-		(net 55)
-		(net_name "/SPI_MOSI_{0}")
+		(net 92)
+		(net_name "Net-(U9-L1)")
 		(layer "F.Cu")
-		(name "$teardrop_padvia$")
-		(hatch none 0.1)
-		(priority 30007)
-		(attr
-			(teardrop
-				(type padvia)
-			)
-		)
+		(name "U9_L1")
+		(hatch edge 0.5)
+		(priority 5)
 		(connect_pads yes
-			(clearance 0)
+			(clearance 0.15)
 		)
-		(min_thickness 0.0254)
+		(min_thickness 0.25)
 		(filled_areas_thickness no)
 		(fill yes
 			(thermal_gap 0.5)
 			(thermal_bridge_width 0.5)
-			(island_removal_mode 1)
-			(island_area_min 10)
 		)
 		(polygon
 			(pts
-				(xy 146.93947 90.35447) (xy 146.73947 90.35447) (xy 146.540274 90.70654) (xy 146.83947 91.46547)
-				(xy 147.138666 90.70654)
+				(xy 169.69947 71.89947) (xy 169.69947 71.40947) (xy 171.40947 71.40947) (xy 172.42947 70.38947)
+				(xy 175.26697 70.38947) (xy 175.41947 70.54197) (xy 175.41947 71.75947) (xy 175.27947 71.89947)
 			)
 		)
@@
 	)
 	(zone
-		(net 3)
-		(net_name "+3V3")
+		(net 51)
+		(net_name "/SPI_SCK_{0}")
 		(layer "F.Cu")
-		(name "U5_3V3")
-		(hatch edge 0.5)
-		(priority 22)
+		(name "$teardrop_padvia$")
+		(hatch none 0.1)
+		(priority 30002)
+		(attr
+			(teardrop
+				(type padvia)
+			)
+		)
 		(connect_pads yes
-			(clearance 0.15)
+			(clearance 0)
 		)
-		(min_thickness 0.25)
+		(min_thickness 0.0254)
 		(filled_areas_thickness no)
 		(fill yes
 			(thermal_gap 0.5)
 			(thermal_bridge_width 0.5)
+			(island_removal_mode 1)
+			(island_area_min 10)
 		)
 		(polygon
 			(pts
-				(xy 150.04447 90.25947) (xy 153.54447 90.25947) (xy 153.54447 94.35947) (xy 150.04447 94.35947)
+				(xy 148.20947 90.35447) (xy 148.00947 90.35447) (xy 147.810274 90.70654) (xy 148.10947 91.46547)
+				(xy 148.408666 90.70654)
 			)
 		)
 	)
 	(zone
-		(net 55)
-		(net_name "/SPI_MOSI_{0}")
+		(net 3)
+		(net_name "+3V3")
 		(layer "F.Cu")
-		(name "$teardrop_padvia$")
-		(hatch none 0.1)
-		(priority 30002)
-		(attr
-			(teardrop
-				(type padvia)
-			)
-		)
+		(name "U5_3V3")
+		(hatch edge 0.5)
+		(priority 22)
 		(connect_pads yes
-			(clearance 0)
+			(clearance 0.15)
 		)
-		(min_thickness 0.0254)
+		(min_thickness 0.25)
 		(filled_areas_thickness no)
 		(fill yes
 			(thermal_gap 0.5)
 			(thermal_bridge_width 0.5)
-			(island_removal_mode 1)
-			(island_area_min 10)
 		)
 		(polygon
 			(pts
-				(xy 146.73947 92.57447) (xy 146.93947 92.57447) (xy 147.138666 92.2224) (xy 146.83947 91.46347)
-				(xy 146.540274 92.2224)
+				(xy 150.04447 90.25947) (xy 153.54447 90.25947) (xy 153.54447 94.35947) (xy 150.04447 94.35947)
 			)
 		)
@@
 	)
 	(zone
-		(net 81)
-		(net_name "/RF_OUT")
+		(net 54)
+		(net_name "/SPI_MISO_{0}")
 		(layer "F.Cu")
 		(name "$teardrop_padvia$")
 		(hatch none 0.1)
-		(priority 30001)
+		(priority 30004)
 		(attr
 			(teardrop
@@
 		(polygon
 			(pts
-				(xy 120.19947 75.65947) (xy 119.84947 75.65947) (xy 119.242739 76.607626) (xy 120.02447 78.46047)
-				(xy 120.806201 76.607626)
+				(xy 149.47947 83.14447) (xy 149.27947 83.14447) (xy 149.080274 83.49654) (xy 149.37947 84.25547)
+				(xy 149.678666 83.49654)
 			)
 		)
 	)
 	(zone
-		(net 3)
-		(net_name "+3V3")
+		(net 81)
+		(net_name "/RF_OUT")
 		(layer "F.Cu")
-		(name "RP2350_3V3")
-		(hatch edge 0.5)
-		(priority 15)
+		(name "$teardrop_padvia$")
+		(hatch none 0.1)
+		(priority 30001)
+		(attr
+			(teardrop
+				(type padvia)
+			)
+		)
 		(connect_pads yes
-			(clearance 0.15)
+			(clearance 0)
 		)
-		(min_thickness 0.25)
+		(min_thickness 0.0254)
 		(filled_areas_thickness no)
 		(fill yes
 			(thermal_gap 0.5)
 			(thermal_bridge_width 0.5)
+			(island_removal_mode 1)
+			(island_area_min 10)
 		)
 		(polygon
 			(pts
-				(xy 157.80947 105.22947) (xy 157.80947 104.82947) (xy 159.10947 104.82947) (xy 159.10947 105.22947)
+				(xy 120.19947 75.65947) (xy 119.84947 75.65947) (xy 119.242739 76.607626) (xy 120.02447 78.46047)
+				(xy 120.806201 76.607626)
 			)
 		)
 	)
 	(zone
-		(net 54)
-		(net_name "/SPI_MISO_{0}")
+		(net 55)
+		(net_name "/SPI_MOSI_{0}")
 		(layer "F.Cu")
 		(name "$teardrop_padvia$")
@@
 		(polygon
 			(pts
-				(xy 149.47947 83.14447) (xy 149.27947 83.14447) (xy 149.080274 83.49654) (xy 149.37947 84.25547)
-				(xy 149.678666 83.49654)
+				(xy 146.93947 90.35447) (xy 146.73947 90.35447) (xy 146.540274 90.70654) (xy 146.83947 91.46547)
+				(xy 147.138666 90.70654)
+			)
+		)
+	)
+	(zone
+		(net 3)
+		(net_name "+3V3")
+		(layer "F.Cu")
+		(name "RP2350_3V3")
+		(hatch edge 0.5)
+		(priority 15)
+		(connect_pads yes
+			(clearance 0.15)
+		)
+		(min_thickness 0.25)
+		(filled_areas_thickness no)
+		(fill yes
+			(thermal_gap 0.5)
+			(thermal_bridge_width 0.5)
+		)
+		(polygon
+			(pts
+				(xy 157.80947 105.22947) (xy 157.80947 104.82947) (xy 159.10947 104.82947) (xy 159.10947 105.22947)
 			)
 		)

Commit message: Finalize working software-defined instrumentation amplifier driver code and signal acquisition, begin prototyping sensor data conversion methods. Add hardware changes needed for expected operation of analog front-end.
Parts:
- U14: value LMV324 -> TLV9144
Connections:
- C37 pad 2: Net-(U12-CAP-) -> unconnected-(C37-Pad2)
- U12 pad 4: Net-(U12-CAP-) -> unconnected-(U12-CAP--Pad4)
Routing:
- added copper zone on B.Cu, net unconnected-(U12-CAP--Pad4)
- removed copper zone on B.Cu, net Net-(U12-CAP-)
Changed lines of the file:
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@@
 	(net 39 "Net-(U11A--)")
 	(net 40 "Net-(U12-CAP+)")
-	(net 41 "Net-(U12-CAP-)")
+	(net 41 "unconnected-(C37-Pad2)")
 	(net 42 "/Software-Defined Instrumentation Amplifier/OUT")
 	(net 43 "/PH_RAW")
@@
 	(net 133 "unconnected-(A1-GPIO17-Pad22)_1")
 	(net 134 "unconnected-(A1-3V3-Pad36)_1")
+	(net 135 "unconnected-(U12-CAP--Pad4)")
 	(footprint "Capacitor_SMD:C_0805_2012Metric_Pad1.18x1.45mm_HandSolder"
 		(layer "F.Cu")
@@
 		(sheetname "/")
 		(sheetfile "LoRa Water Quality Management System Sensor Node.kicad_sch")
-		(attr through_hole)
+		(attr through_hole dnp)
 		(fp_line
 			(start 10.61 22.65)
@@
 			)
 		)
-		(property "Value" "LMV324"
+		(property "Value" "TLV9144"
 			(at 0 3.45 0)
 			(layer "F.Fab")
@@
 			(size 1.8288 0.5334)
 			(layers "B.Cu" "B.Mask" "B.Paste")
-			(net 41 "Net-(U12-CAP-)")
+			(net 135 "unconnected-(U12-CAP--Pad4)")
 			(pinfunction "CAP-")
 			(pintype "input")
@@
 			(layers "B.Cu" "B.Mask" "B.Paste")
 			(roundrect_rratio 0.188679)
-			(net 41 "Net-(U12-CAP-)")
+			(net 41 "unconnected-(C37-Pad2)")
 			(pintype "passive")
 		)
@@
 	)
 	(zone
-		(net 41)
-		(net_name "Net-(U12-CAP-)")
+		(net 135)
+		(net_name "unconnected-(U12-CAP--Pad4)")
 		(layer "B.Cu")
 		(name "SWCAP-")

Commit message: Add finalized firmware - implemented power savings mode and implemented complete FSM.
Parts:
- R35, R36, R37, R38: value 10k -> 3.3M
Changed lines of the file:
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@@
 			)
 		)
-		(property "Value" "10k"
+		(property "Value" "3.3M"
 			(at 0 1.65 0)
 			(layer "F.Fab")
@@
 			)
 		)
-		(property "Value" "10k"
+		(property "Value" "3.3M"
 			(at 0 1.65 0)
 			(layer "F.Fab")
@@
 			)
 		)
-		(property "Value" "10k"
+		(property "Value" "3.3M"
 			(at 0 1.65 0)
 			(layer "F.Fab")
@@
 			)
 		)
-		(property "Value" "10k"
+		(property "Value" "3.3M"
 			(at 0 1.65 0)
 			(layer "F.Fab")
