File: Sensor Node/receiver/lwqms_receiver/lwqms_receiver.kicad_pcb (KiCad board)
At the start: 2 copper layers, 58 x 102 mm, 18 parts, among them J1 Conn_01x20, J2 Conn_01x20, SW1 Tactile Pushbutton, U1 Core1262 HF

Commit message: Add receiver gerber files and updated testing CSVs.
Other:
- board text added: "Designed by Matthew Sharp"
Changed lines of the file:
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@@
 			(outputformat 1)
 			(mirror no)
-			(drillshape 1)
+			(drillshape 0)
 			(scaleselection 1)
-			(outputdirectory "")
+			(outputdirectory "gerbers/")
 		)
 	)
@@
 			)
 			(justify left bottom)
+		)
+	)
+	(gr_text "Designed by Matthew Sharp"
+		(at 113 117 90)
+		(layer "F.Cu")
+		(effects
+			(font
+				(size 1.2 1.2)
+				(thickness 0.15)
+			)
+			(justify left bottom)
